File: KiCad_M644_breakout_v1.2d/M644_breakout_v1.2d.kicad_pcb (KiCad board)
At the start: 2 copper layers, 54.6 x 45 mm, 62 parts, among them IC1 ATMEGA16/32/644/1284, IC2 78TV, Q1 16Mhz, SW1/PC5 SMD_TACT_4x4, X2 DG300-5.0-02P-12

Commit message: Slightly edited the pics and pcb hardware board
Parts:
- added REF**: Pin_Header_Straight_2x04_Pitch2.54mm, Pin_Headers:Pin_Header_Straight_2x04_Pitch2.54mm, F.Cu at (172.0, 117.3)
- added REF**: Pin_Header_Straight_1x04_Pitch2.54mm, Pin_Headers:Pin_Header_Straight_1x04_Pitch2.54mm, F.Cu at (174.5, 91.9)
- moved JP11 2.84 mm to (155.5, 97.0)
- moved JP5 2.84 mm to (152.9, 97.0)
- moved JP4 2.84 mm to (150.4, 97.0)
- moved JP12 1.80 mm to (155.5, 94.5)
- moved JP6 1.80 mm to (152.9, 94.5)
- moved JP7 1.80 mm to (150.4, 94.5)
- moved JP1 1.27 mm to (140.2, 86.9)
- moved JP13 1.27 mm to (155.5, 91.9)
- moved JP27 1.27 mm to (127.5, 107.2)
- moved JP28 1.27 mm to (127.5, 117.3)
- moved JP9 1.27 mm to (152.9, 91.9)
- moved SW1/PC5 1.27 mm to (132.6, 91.9)
- moved JP8 1.27 mm to (150.4, 91.9)
Routing:
- net VCC: track 224.0 -> 232.6 mm
- net /MISO: track 21.7 -> 27.2 mm, vias 0 -> 1
- net /MOSI: track 29.2 -> 33.7 mm, vias 0 -> 1
- net /PB3: track 14.9 -> 13.6 mm
- net /PA3: track 17.8 -> 16.5 mm
- net /PC4: track 14.6 -> 15.8 mm
- net Net-(R3-PadP$1): track 9.37 -> 10.6 mm
- net /PA1: track 15.9 -> 14.6 mm
- net /PA0: track 15.3 -> 14.0 mm
- net /PB2: track 15.0 -> 13.7 mm
- net /PA2: track 16.8 -> 15.5 mm
- net /PB0: track 16.5 -> 15.2 mm
- net /PB1: track 15.5 -> 14.2 mm
- net /PB4: track 15.3 -> 14.1 mm
- net GND: track 247.0 -> 247.6 mm
Other:
- board size 54.6 x 45 mm -> 54.9 x 45 mm

Commit message: Added new factory design 1.2d-a
Routing:
- net /PC6: track 25.9 -> 24.6 mm
- net /PC3: track 17.1 -> 16.3 mm
- net /PC2: track 15.9 -> 15.3 mm
- net GND: vias 10 -> 55
- net N$9: vias 1 -> 0
- net N$8: vias 1 -> 0
- net N$7: vias 1 -> 0
- net (no net): vias 0 -> 3
- added copper zone on F.Cu, net GND
Other:
- board text added: "RX0"
- board text added: "RX1"
- board text added: "SCL"
- board text added: "SDA"
- board text added: "TX0"
- board text added: "TX1"
- board text added: "XCK0"
- board text added: "XCK1"
- board text removed: "rx0"
- board text removed: "rx1"
- board text removed: "scl"
- board text removed: "sda"
- board text removed: "tx0"
- board text removed: "tx1"
- board text removed: "xck0"
- board text removed: "xck1"

Commit message: Updated PCB design
Routing:
- net /PD7: track 15.4 -> 14.7 mm
Changed lines of the file:
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@@
     (thickness 1.6)
     (drawings 118)
-    (tracks 548)
+    (tracks 545)
     (zones 0)
     (modules 64)
@@
   )
   (setup
-    (last_trace_width 0.25)
+    (last_trace_width 0.4064)
     (user_trace_width 0.4064)
     (user_trace_width 0.6096)
@@
   (segment (start 137.7061 123.6936) (end 141.1097 113.5336) (width 0.4064) (layer Bottom) (net 25))
   (segment (start 137.7061 124.9636) (end 137.7061 123.6936) (width 0.4064) (layer Bottom) (net 25))
-  (segment (start 140.2461 124.9636) (end 140.2461 122.4236) (width 0.4064) (layer Bottom) (net 26))
-  (segment (start 140.2461 122.4236) (end 141.5161 121.1536) (width 0.4064) (layer Bottom) (net 26))
-  (segment (start 141.5161 121.1536) (end 142.7493 121.172) (width 0.4064) (layer Bottom) (net 26))
-  (segment (start 142.7493 121.172) (end 143.0438 120.9843) (width 0.4064) (layer Bottom) (net 26))
-  (segment (start 143.0438 120.9843) (end 143.0701 120.9255) (width 0.4064) (layer Bottom) (net 26))
-  (segment (start 143.0701 120.9255) (end 144.0561 117.3436) (width 0.4064) (layer Bottom) (net 26))
   (segment (start 144.0561 117.3436) (end 144.0561 114.0162) (width 0.4064) (layer Bottom) (net 26))
   (segment (start 144.0561 114.0162) (end 143.5989 113.0256) (width 0.4064) (layer Bottom) (net 26))
   (segment (start 143.5989 113.0256) (end 143.5861 111.7136) (width 0.4064) (layer Bottom) (net 26))
+  (segment (start 140.2461 123.178487) (end 143.286987 120.1376) (width 0.4064) (layer Bottom) (net 26))
+  (segment (start 140.2461 124.9636) (end 140.2461 123.178487) (width 0.4064) (layer Bottom) (net 26))
+  (segment (start 143.286987 120.1376) (end 144.0561 117.3436) (width 0.4064) (layer Bottom) (net 26))
   (segment (start 144.4117 112.9748) (end 144.3861 111.7136) (width 0.4064) (layer Bottom) (net 27))
   (segment (start 144.7419 113.5336) (end 144.4117 112.9748) (width 0.4064) (layer Bottom) (net 27))
